Commit message: Update turtlebot3_waffle_pi.urdf.xacro

File: turtlebot3/turtlebot3_description/urdf/turtlebot3_waffle_pi.urdf.xacro (robot description, xacro)
@@ -35,10 +35,10 @@
     <parent link="base_link"/>
     <child link="wheel_left_link"/>
-    <origin xyz="-0.094 0.065 0.035" rpy="0 0 0"/>
+    <origin xyz="-0.094 0.065 0.035" rpy="-1.57 0 0"/>
     <axis xyz="0 0 1"/>
   </joint>
   <link name="wheel_left_link">
     <visual>
-      <origin xyz="0 0 0" rpy="0 0 0"/>
+      <origin xyz="0 0 0" rpy="1.57 0 0"/>
       <geometry>
         <mesh filename="package://turtlebot3_description/meshes/wheels/left_tire.stl" scale="0.001 0.001 0.001"/>
@@ -63,10 +63,10 @@
     <parent link="base_link"/>
     <child link="wheel_right_link"/>
-    <origin xyz="-0.094 -0.065 0.035" rpy="0 0 0"/>
+    <origin xyz="-0.094 -0.065 0.035" rpy="-1.57 0 0"/>
     <axis xyz="0 0 1"/>
   </joint>
   <link name="wheel_right_link">
     <visual>
-      <origin xyz="0 0 0" rpy="0 0 0"/>
+      <origin xyz="0 0 0" rpy="1.57 0 0"/>
       <geometry>
         <mesh filename="package://turtlebot3_description/meshes/wheels/right_tire.stl" scale="0.001 0.001 0.001"/>

Commit message: modify : cjw_recommit_by_cej

File: turtlebot3/turtlebot3_description/urdf/turtlebot3_waffle_pi.urdf.xacro (robot description, xacro)
@@ -7,9 +7,9 @@
     <parent link="base_footprint"/>
     <child link="base_link" />
-    <origin xyz="0 0 0.0" rpy="0 0 0"/>
+    <origin xyz="0 0 0" rpy="0 0 0"/>
   </joint>
   <link name="base_link">
     <visual>
-      <origin xyz="-0.064 0 0.055" rpy="0 0 0"/>
+      <origin xyz="-0.064 0 0.055" rpy="0 0 0"/> <!--<origin xyz="-0.064 0 0.055" rpy="0 0 0"/>-->
       <geometry>
         <box size="0.210 0.145 0.01"/>
@@ -19,12 +19,12 @@
     </visual>
     <collision>
-      <origin xyz="-0.064 0 0.047" rpy="0 0 0"/>
+      <origin xyz="-0.064 0 0.055" rpy="0 0 0"/> <!--<origin xyz="-0.064 0 0.055" rpy="0 0 0"/>-->
       <geometry>
-        <box size="0.145 0.210 0.094"/>
+        <box size="0.210 0.145 0.01"/>
       </geometry>
     </collision>
     <inertial>
       <origin xyz="0 0 0" rpy="0 0 0"/>
-      <mass value="1.3729096e+00"/>
+      <mass value="1.3729096e+00"/> <!-- mass value="1.3729096e+00"-->
       <inertia ixx="8.7002718e-03" ixy="-4.7576583e-05" ixz="1.1160499e-04"
                iyy="8.6195418e-03" iyz="-3.5422299e-06"
@@ -35,5 +35,5 @@
     <parent link="base_link"/>
     <child link="wheel_left_link"/>
-    <origin xyz="-0.094 0.065 0.035" rpy="-1.57 0 0"/>
+    <origin xyz="-0.094 0.065 0.035" rpy="-1.57 0 0"/><!-- xyz="-0.094 0.065 0.035"-->
     <axis xyz="0 0 1"/>
   </joint>
@@ -49,10 +49,10 @@
       <origin xyz="0 0 0" rpy="0 0 0"/>
       <geometry>
-        <cylinder length="0.025" radius="0.067"/>
+        <cylinder length="0.025" radius="0.0335"/>
       </geometry>
     </collision>
     <inertial>
       <origin xyz="0 0 0" />
-      <mass value="2.8498940e-02" />
+      <mass value="2.8498940e-02" /> <!-- 2.8498940e-02-->
       <inertia ixx="1.1175580e-05" ixy="-4.2369783e-11" ixz="-5.9381719e-09"
                iyy="1.1192413e-05" iyz="-1.4400107e-11"
@@ -63,5 +63,5 @@
     <parent link="base_link"/>
     <child link="wheel_right_link"/>
-    <origin xyz="-0.094 -0.065 0.035" rpy="-1.57 0 0"/>
+    <origin xyz="-0.094 -0.065 0.035" rpy="-1.57 0 0"/> <!--xyz="-0.094 -0.065 0.035"-->
     <axis xyz="0 0 1"/>
   </joint>
@@ -77,10 +77,10 @@
       <origin xyz="0 0 0" rpy="0 0 0"/>
       <geometry>
-        <cylinder length="0.025" radius="0.067"/>
+        <cylinder length="0.025" radius="0.0335"/>
       </geometry>
     </collision>
     <inertial>
       <origin xyz="0 0 0" />
-      <mass value="2.8498940e-02" />
+      <mass value="2.8498940e-02" /> <!-- 2.8498940e-02-->
       <inertia ixx="1.1175580e-05" ixy="-4.2369783e-11" ixz="-5.9381719e-09"
                iyy="1.1192413e-05" iyz="-1.4400107e-11"
@@ -88,13 +88,13 @@
       </inertial>
   </link>
-  <joint name="caster_back_right_joint" type="fixed">
+  <joint name="caster_back_right_joint" type="continuous"> <!--type="fixed"-->
     <parent link="base_link"/>
     <child link="caster_back_right_link"/>
-    <origin xyz="0.02 0.0 0.035" rpy="-1.57 0 0"/>
+    <origin xyz="0.02 0.0 0.035" rpy="-1.57 0 0"/><!--xyz="0.02 0.0 0.035"-->
   </joint>
   <link name="caster_back_right_link">
     <visual>
         <geometry>
-        <cylinder radius="0.03" length="0.01"/>
+        <cylinder radius="0.0335" length="0.025"/> <!--<cylinder radius="0.03" length="0.01"/>-->
         </geometry>
       <origin xyz="0 0 0" rpy="0 0 0"/>
@@ -104,10 +104,10 @@
       <origin xyz="0 0.001 0" rpy="0 0 0"/>
       <geometry>
-        <box size="0.030 0.009 0.020"/>
+        <cylinder radius="0.0335" length="0.025"/> <!--box size="0.030 0.009 0.020"-->
       </geometry>
     </collision>
     <inertial>
       <origin xyz="0 0 0" />
-      <mass value="0.005" />
+      <mass value="2.8498940e-04" />
       <inertia ixx="0.001" ixy="0.0" ixz="0.0"
                iyy="0.001" iyz="0.0"
@@ -115,4 +115,5 @@
     </inertial>
   </link>
+<!--
   <joint name="caster_back_left_joint" type="fixed">
     <parent link="base_link"/>
@@ -135,4 +136,5 @@
     </inertial>
   </link>
+-->
   <joint name="imu_joint" type="fixed">
     <parent link="base_link"/>

Commit message: modify : cjw_recommit_by_cej
error path

File: turtlebot3/turtlebot3_description/urdf/turtlebot3_waffle_pi.urdf.xacro (robot description, xacro)
@@ -7,9 +7,10 @@
     <parent link="base_footprint"/>
     <child link="base_link" />
-    <origin xyz="0 0 0.0" rpy="0 0 0"/>
+    <origin xyz="0 0 0" rpy="0 0 0"/>
   </joint>
+ <!--minipjt_modify-->
   <link name="base_link">
     <visual>
-      <origin xyz="-0.064 0 0.055" rpy="0 0 0"/>
+      <origin xyz="-0.064 0 0.055" rpy="0 0 0"/> <!--<origin xyz="-0.064 0 0.055" rpy="0 0 0"/>-->
       <geometry>
         <box size="0.210 0.145 0.01"/>
@@ -19,12 +20,12 @@
     </visual>
     <collision>
-      <origin xyz="-0.064 0 0.047" rpy="0 0 0"/>
+      <origin xyz="-0.064 0 0.055" rpy="0 0 0"/> <!--<origin xyz="-0.064 0 0.055" rpy="0 0 0"/>-->
       <geometry>
-        <box size="0.145 0.210 0.094"/>
+        <box size="0.210 0.145 0.01"/>
       </geometry>
     </collision>
     <inertial>
       <origin xyz="0 0 0" rpy="0 0 0"/>
-      <mass value="1.3729096e+00"/>
+      <mass value="1.3729096e+00"/> <!-- mass value="1.3729096e+00"-->
       <inertia ixx="8.7002718e-03" ixy="-4.7576583e-05" ixz="1.1160499e-04"
                iyy="8.6195418e-03" iyz="-3.5422299e-06"
@@ -35,5 +36,5 @@
     <parent link="base_link"/>
     <child link="wheel_left_link"/>
-    <origin xyz="-0.094 0.065 0.035" rpy="-1.57 0 0"/>
+    <origin xyz="-0.094 0.065 0.035" rpy="-1.57 0 0"/><!-- xyz="-0.094 0.065 0.035"-->
     <axis xyz="0 0 1"/>
   </joint>
@@ -49,10 +50,10 @@
       <origin xyz="0 0 0" rpy="0 0 0"/>
       <geometry>
-        <cylinder length="0.025" radius="0.067"/>
+        <cylinder length="0.025" radius="0.0335"/>
       </geometry>
     </collision>
     <inertial>
       <origin xyz="0 0 0" />
-      <mass value="2.8498940e-02" />
+      <mass value="2.8498940e-02" /> <!-- 2.8498940e-02-->
       <inertia ixx="1.1175580e-05" ixy="-4.2369783e-11" ixz="-5.9381719e-09"
                iyy="1.1192413e-05" iyz="-1.4400107e-11"
@@ -63,5 +64,5 @@
     <parent link="base_link"/>
     <child link="wheel_right_link"/>
-    <origin xyz="-0.094 -0.065 0.035" rpy="-1.57 0 0"/>
+    <origin xyz="-0.094 -0.065 0.035" rpy="-1.57 0 0"/> <!--xyz="-0.094 -0.065 0.035"-->
     <axis xyz="0 0 1"/>
   </joint>
@@ -77,10 +78,10 @@
       <origin xyz="0 0 0" rpy="0 0 0"/>
       <geometry>
-        <cylinder length="0.025" radius="0.067"/>
+        <cylinder length="0.025" radius="0.0335"/>
       </geometry>
     </collision>
     <inertial>
       <origin xyz="0 0 0" />
-      <mass value="2.8498940e-02" />
+      <mass value="2.8498940e-02" /> <!-- 2.8498940e-02-->
       <inertia ixx="1.1175580e-05" ixy="-4.2369783e-11" ixz="-5.9381719e-09"
                iyy="1.1192413e-05" iyz="-1.4400107e-11"
@@ -88,13 +89,13 @@
       </inertial>
   </link>
-  <joint name="caster_back_right_joint" type="fixed">
+  <joint name="caster_back_right_joint" type="continuous"> <!--type="fixed"-->
     <parent link="base_link"/>
     <child link="caster_back_right_link"/>
-    <origin xyz="0.02 0.0 0.035" rpy="-1.57 0 0"/>
+    <origin xyz="0.02 0.0 0.035" rpy="-1.57 0 0"/><!--xyz="0.02 0.0 0.035"-->
   </joint>
   <link name="caster_back_right_link">
     <visual>
         <geometry>
-        <cylinder radius="0.03" length="0.01"/>
+        <cylinder radius="0.0335" length="0.025"/> <!--<cylinder radius="0.03" length="0.01"/>-->
         </geometry>
       <origin xyz="0 0 0" rpy="0 0 0"/>
@@ -104,10 +105,10 @@
       <origin xyz="0 0.001 0" rpy="0 0 0"/>
       <geometry>
-        <box size="0.030 0.009 0.020"/>
+        <cylinder radius="0.0335" length="0.025"/> <!--box size="0.030 0.009 0.020"-->
       </geometry>
     </collision>
     <inertial>
       <origin xyz="0 0 0" />
-      <mass value="0.005" />
+      <mass value="2.8498940e-04" />
       <inertia ixx="0.001" ixy="0.0" ixz="0.0"
                iyy="0.001" iyz="0.0"
@@ -115,4 +116,5 @@
     </inertial>
   </link>
+<!--
   <joint name="caster_back_left_joint" type="fixed">
     <parent link="base_link"/>
@@ -135,4 +137,5 @@
     </inertial>
   </link>
+-->
   <joint name="imu_joint" type="fixed">
     <parent link="base_link"/>

Commit message: add : 20240320

File: turtlebot3/turtlebot3_description/urdf/turtlebot3_waffle_pi.urdf.xacro (robot description, xacro)
@@ -7,25 +7,24 @@
     <parent link="base_footprint"/>
     <child link="base_link" />
-    <origin xyz="0 0 0" rpy="0 0 0"/>
+    <origin xyz="0 0 0.010" rpy="0 0 0"/>
   </joint>
- <!--minipjt_modify-->
   <link name="base_link">
     <visual>
-      <origin xyz="-0.064 0 0.055" rpy="0 0 0"/> <!--<origin xyz="-0.064 0 0.055" rpy="0 0 0"/>-->
+      <origin xyz="-0.064 0 0.055" rpy="0 0 0"/>
       <geometry>
         <box size="0.210 0.145 0.01"/>
-        <mesh filename="package://turtlebot3_description/meshes/bases/waffle_pi_base.stl" scale="0.001 0.001 0.001"/>
+        <!--<mesh filename="package://turtlebot3_description/meshes/bases/waffle_pi_base.stl" scale="0.001 0.001 0.001"/>-->
       </geometry>
       <material name="light_black"/>
     </visual>
     <collision>
-      <origin xyz="-0.064 0 0.055" rpy="0 0 0"/> <!--<origin xyz="-0.064 0 0.055" rpy="0 0 0"/>-->
+      <origin xyz="-0.064 0 0.055" rpy="0 0 0"/> <!--xyz="-0.064 0 0.047"-->
       <geometry>
-        <box size="0.210 0.145 0.01"/>
+        <box size="0.21 0.145 0.01"/>
       </geometry>
     </collision>
     <inertial>
       <origin xyz="0 0 0" rpy="0 0 0"/>
-      <mass value="1.3729096e+00"/> <!-- mass value="1.3729096e+00"-->
+      <mass value="1.3729096e+00"/>
       <inertia ixx="8.7002718e-03" ixy="-4.7576583e-05" ixz="1.1160499e-04"
                iyy="8.6195418e-03" iyz="-3.5422299e-06"
@@ -36,5 +35,5 @@
     <parent link="base_link"/>
     <child link="wheel_left_link"/>
-    <origin xyz="-0.094 0.065 0.035" rpy="-1.57 0 0"/><!-- xyz="-0.094 0.065 0.035"-->
+    <origin xyz="-0.0 0.065 0.035" rpy="-1.57 0 0"/> <!--xyz="0.0 0.144 0.023"-->
     <axis xyz="0 0 1"/>
   </joint>
@@ -50,10 +49,10 @@
       <origin xyz="0 0 0" rpy="0 0 0"/>
       <geometry>
-        <cylinder length="0.025" radius="0.0335"/>
+        <cylinder length="0.025" radius="0.0335"/><!--<cylinder length="0.018" radius="0.033"/>-->
       </geometry>
     </collision>
     <inertial>
       <origin xyz="0 0 0" />
-      <mass value="2.8498940e-02" /> <!-- 2.8498940e-02-->
+      <mass value="2.8498940e-02" />
       <inertia ixx="1.1175580e-05" ixy="-4.2369783e-11" ixz="-5.9381719e-09"
                iyy="1.1192413e-05" iyz="-1.4400107e-11"
@@ -64,5 +63,5 @@
     <parent link="base_link"/>
     <child link="wheel_right_link"/>
-    <origin xyz="-0.094 -0.065 0.035" rpy="-1.57 0 0"/> <!--xyz="-0.094 -0.065 0.035"-->
+    <origin xyz="-0.0 -0.065 0.035" rpy="-1.57 0 0"/>
     <axis xyz="0 0 1"/>
   </joint>
@@ -78,10 +77,10 @@
       <origin xyz="0 0 0" rpy="0 0 0"/>
       <geometry>
-        <cylinder length="0.025" radius="0.0335"/>
+        <cylinder length="0.025" radius="0.0335"/> <!--<cylinder length="0.018" radius="0.033"/>-->
       </geometry>
     </collision>
     <inertial>
       <origin xyz="0 0 0" />
-      <mass value="2.8498940e-02" /> <!-- 2.8498940e-02-->
+      <mass value="2.8498940e-02" />
       <inertia ixx="1.1175580e-05" ixy="-4.2369783e-11" ixz="-5.9381719e-09"
                iyy="1.1192413e-05" iyz="-1.4400107e-11"
@@ -89,26 +88,26 @@
       </inertial>
   </link>
-  <joint name="caster_back_right_joint" type="continuous"> <!--type="fixed"-->
+  <joint name="caster_back_right_joint" type="fixed">
     <parent link="base_link"/>
     <child link="caster_back_right_link"/>
-    <origin xyz="0.02 0.0 0.035" rpy="-1.57 0 0"/><!--xyz="0.02 0.0 0.035"-->
+    <origin xyz="-0.177 -0.064 -0.004" rpy="-1.57 0 0"/> <!--<origin xyz="-0.177 -0.064 -0.004" rpy="-1.57 0 0"/>-->
   </joint>
   <link name="caster_back_right_link">
-    <visual>
-        <geometry>
-        <cylinder radius="0.0335" length="0.025"/> <!--<cylinder radius="0.03" length="0.01"/>-->
-        </geometry>
-      <origin xyz="0 0 0" rpy="0 0 0"/>
-      <material name="grey"/>
+      <visual>
+      <origin xyz="0.05 -0.0295 0.065" rpy="1.57 0 0"/>
+      <geometry>
+        <mesh filename="package://turtlebot3_description/meshes/wheels/right_tire.stl" scale="0.001 0.001 0.001"/>
+      </geometry>
+      <material name="dark"/>
     </visual>
     <collision>
       <origin xyz="0 0.001 0" rpy="0 0 0"/>
       <geometry>
-        <cylinder radius="0.0335" length="0.025"/> <!--box size="0.030 0.009 0.020"-->
+        <box size="0.030 0.009 0.020"/>
       </geometry>
     </collision>
     <inertial>
       <origin xyz="0 0 0" />
-      <mass value="2.8498940e-04" />
+      <mass value="0.005" />
       <inertia ixx="0.001" ixy="0.0" ixz="0.0"
                iyy="0.001" iyz="0.0"
@@ -116,9 +115,8 @@
     </inertial>
   </link>
-<!--
   <joint name="caster_back_left_joint" type="fixed">
     <parent link="base_link"/>
     <child link="caster_back_left_link"/>
-    <origin xyz="0.02 0.00 0.03" rpy="-1.57 0 0"/>
+    <origin xyz="-0.177 0.064 -0.004" rpy="-1.57 0 0"/>
   </joint>
   <link name="caster_back_left_link">
@@ -137,9 +135,8 @@
     </inertial>
   </link>
--->
   <joint name="imu_joint" type="fixed">
     <parent link="base_link"/>
     <child link="imu_link"/>
-    <origin xyz="0.0 0 0.01" rpy="0 0 0"/>
+    <origin xyz="0.0 0 0.068" rpy="0 0 0"/>
   </joint>
   <link name="imu_link"/>
@@ -147,5 +144,5 @@
     <parent link="base_link"/>
     <child link="base_scan"/>
-    <origin xyz="-0.064 0 0.1" rpy="0 0 0"/>
+    <origin xyz="-0.064 0 0.122" rpy="0 0 0"/>
   </joint>
   <link name="base_scan">
@@ -172,5 +169,5 @@
   </link>
   <joint name="camera_joint" type="fixed">
-    <origin xyz="0.073 -0.011 0.034" rpy="0 0 0"/>
+    <origin xyz="0.073 -0.011 0.084" rpy="0 0 0"/>
     <parent link="base_link"/>
     <child link="camera_link"/>
